File: pcb/adelheid.sch (KiCad schematic (older format))
At the start: 40 parts, among them J1 USB_B_Mini, J12 VCC, J13 D+, J14 D-, J15 GND, J2 MISO, J3 VCC, J4 SCK, J5 MOSI, J6 RES, J7 GND, J8 PF4, J9 PF5, Q1 2N7002, U1 USBLC6-2SC6, U2 ATmega32U4-AU, Y1 Crystal_GND24

Commit message: added encoder
Parts:
- removed J8: PF4, Pin_Headers:Pin_Header_Straight_1x01_Pitch2.54mm, symbol Connector_Generic:Conn_01x01
- removed J9: PF5, Pin_Headers:Pin_Header_Straight_1x01_Pitch2.54mm, symbol Connector_Generic:Conn_01x01
- C1, C2, C3, C4, C5, C6, C7, C8, C9: symbol Device:C -> adelheid-rescue:C-Device
- H1, H2, H3, H4, H5, H6, H7, H8: symbol Mechanical:MountingHole -> adelheid-rescue:MountingHole-Mechanical
- J1: symbol Connector:USB_B_Micro -> adelheid-rescue:USB_B_Micro-Connector
- J12, J13, J14, J15, J2, J3, J4, J5, J6, J7: symbol Connector_Generic:Conn_01x01 -> adelheid-rescue:Conn_01x01-Connector_Generic
- Q1: symbol Transistor_FET:2N7002 -> adelheid-rescue:2N7002-Transistor_FET
- R1, R2, R3, R4, R5: symbol Device:R -> adelheid-rescue:R-Device
- SWR1: symbol Switch:SW_Push -> adelheid-rescue:SW_Push-Switch
- Y1: symbol Device:Crystal_GND24 -> adelheid-rescue:Crystal_GND24-Device
Connections:
- wire segments 143 -> 145
Other:
- note added: "PF4"
- note added: "PF5\n"
