File: pcb/matrix.sch (KiCad schematic (older format))
At the start: 281 parts

Commit message: added encoder
Parts:
- removed MX72: MX-LED, ai03-MX_only:MXOnly-1U, symbol ai03-schematic_library:MX-LED
- removed RL72: R, Resistor_SMD:R_0805_2012Metric_Pad1.15x1.40mm_HandSolder, symbol Device:R
- added U3: rotary_encoder, encoder:RotaryEncoder_Alps_EC11E-Switch_Vertical_H20mm, symbol New_Library:rotary_encoder
- D1, D10, D11, D12, D13, D14, D15, D16, D17, D18, D19, D2, D20, D21, D22, D23, D24, D25, D26, D27, D28, D29, D3, D30, D31, D32, D33, D34, D35, D36, D37, D38, D39, D4, D40, D41, D42, D43, D44, D45, D46, D47, D48, D49, D5, D50, D51, D52, D53, D54, D55, D56, D57, D58, D59, D6, D60, D61, D62, D63, D64, D65, D66, D67, D68, D69, D7, D70, D71, D72, D73, D74, D75, D76, D77, D78, D79, D8, D80, D81, D82, D9: symbol Device:D -> adelheid-rescue:D-Device
- LS1, LS10, LS11, LS12, LS13, LS14, LS15, LS16, LS17, LS2, LS3, LS4, LS5, LS6, LS7, LS8, LS9: symbol Device:LED -> adelheid-rescue:LED-Device
- RL1, RL10, RL11, RL12, RL13, RL14, RL15, RL16, RL17, RL18, RL19, RL2, RL20, RL21, RL22, RL23, RL24, RL25, RL26, RL27, RL28, RL29, RL3, RL30, RL31, RL32, RL33, RL34, RL35, RL36, RL37, RL38, RL39, RL4, RL40, RL41, RL42, RL43, RL44, RL45, RL46, RL47, RL48, RL49, RL5, RL50, RL51, RL52, RL53, RL54, RL55, RL56, RL57, RL58, RL59, RL6, RL60, RL61, RL62, RL63, RL64, RL65, RL66, RL67, RL68, RL69, RL7, RL70, RL71, RL73, RL74, RL75, RL76, RL77, RL78, RL79, RL8, RL80, RL81, RL82, RL9, RS1, RS10, RS11, RS12, RS13, RS14, RS15, RS16, RS17, RS2, RS3, RS4, RS5, RS6, RS7, RS8, RS9: symbol Device:R -> adelheid-rescue:R-Device
Connections:
- net labels added: GND-power, PF4, PF5
- wire segments 854 -> 860
